File: Makerspace_THT_Workshop/Makerspace_THT_Workshop.kicad_pcb (KiCad board)
At the start: 2 copper layers, 135.6 x 104.2 mm, 24 parts, among them SW1 SW_SPDT, U1 LM358, U2 LMC555xN

Commit message: Updated PCB with testpoints and text
Parts:
- moved G*** 0.40 mm to (131.8, 113.5)
- moved G*** 0.20 mm to (147.6, 132.4)
Routing:
- net Net-(U2-TR): track 65.9 -> 66.6 mm
Other:
- board text added: "Designed by: Austin Nguyen"
- board text added: "Dino Sniffer Voltage Detecting Dino V1.0"
- board text removed: "Dino Sniffer"
- board text removed: "Voltage Detecting Dino V1.0"
